Commit message: new packages
-susag_nav2(slam_toolbox  and Nav2)
-susag_cartographer
-susag_bringup(still buidling it)
modified the urdf plugins for the appropriate gazebo and ros version

laste tesed and working version tested on 21/09/25

File: src/susag_robot_description/urdf/susag_robot.xacro (robot description, xacro)
@@ -113,4 +113,5 @@
   <collision>
     <origin xyz="0.21 -0.3 -0.1" rpy="0 0 0"/>
+    <origin xyz="0.21 -0.3 -0.1" rpy="0 0 0"/>
     <geometry>
       <mesh filename="file://$(find susag_robot_description)/meshes/left_wheel_back_1.stl" scale="0.001 0.001 0.001"/>
@@ -158,4 +159,13 @@
   </collision>
 </link>
+<!-- Optical frame for rgbd camera (REP-103/120: x-right, y-down, z-forward) -->
+<link name="rgbdcam_1_optical"/>
+<joint name="rgbdcam_1_optical_joint" type="fixed">
+  <parent link="rgbdcam_1"/>
+  <child link="rgbdcam_1_optical"/>
+  <!-- Position this at the optical center of the sensor.
+       Start with zero offset, then tune xyz as needed. -->
+  <origin xyz="0 0 0" rpy="-1.570796 0 -1.570796"/>
+</joint>
 <joint name="right_wheel_back_joint" type="continuous">
   <origin xyz="-0.21 -0.3 0.1" rpy="0 0 0"/>
